Commit message: chore : - add new world included launch file - add robot and launch file - modified urdf robot and setup.py

File: urdf/medical_delivery.xacro (robot description, xacro)
@@ -444,4 +444,20 @@
   </collision>
 </link>
+<link name="imu_link">
+  <visual>
+    <geometry>
+      <box size="0.02 0.02 0.01"/>
+    </geometry>
+  </visual>
+  <collision>
+    <geometry>
+      <box size="0.02 0.02 0.01"/>
+    </geometry>
+  </collision>
+  <inertial>
+    <mass value="0.01"/>
+    <inertia ixx="1e-5" ixy="0" ixz="0" iyy="1e-5" iyz="0" izz="1e-5"/>
+  </inertial>
+</link>
 <link name="lidar_camera_1">
   <inertial>
@@ -464,4 +480,5 @@
   </collision>
 </link>
+<link name="camera_depth_optical_frame"/>
 <link name="camera_base_1">
   <inertial>
@@ -471,5 +488,5 @@
   </inertial>
   <visual>
-    <origin xyz="0.0 -0.30199 -0.238833" rpy="0 0 0"/>
+    <origin xyz="-0.30199 0 -0.238833" rpy="0 0 -1.570796"/>
     <geometry>
       <mesh filename="file://$(find medical_delivery_robot)/meshes/camera_base_1.stl" scale="0.001 0.001 0.001"/>
@@ -745,7 +762,17 @@
 </joint>
 <joint name="Rigid 36" type="fixed">
-  <origin xyz="-0.240313 0.362521 0.033" rpy="0 0 0"/>
+  <origin xyz="-0.240313 0.362521 0.033" rpy="0 0 1.570796"/>
   <parent link="top_cover_body_1"/>
   <child link="camera_base_1"/>
+</joint>
+<joint name="camera_depth_optical_joint" type="fixed">
+  <parent link="camera_base_1"/>
+  <child link="camera_depth_optical_frame"/>
+  <origin xyz="0 0 0" rpy="-1.570796 0 -1.570796"/>
+</joint>
+<joint name="imu_joint" type="fixed">
+  <parent link="base_link"/>
+  <child link="imu_link"/>
+  <origin xyz="0 0 0.1" rpy="0 0 0"/>
 </joint>
 <joint name="Rigid 37" type="fixed">

Commit message: Improves robot URDF and obstacle avoidance logic
Refines robot model by correcting wheel and joint placements, updating
IMU and caster wheel positions, and adjusting base orientation for better
simulation accuracy. Updates obstacle avoidance logic for more concise
code and lowers the minimum safe distance for improved navigation.
Enhances future maintainability and aligns physical model with expected
behavior.

File: urdf/medical_delivery.xacro (robot description, xacro)
@@ -11,5 +11,5 @@
   </inertial>
   <visual>
-    <origin xyz="0 0 0" rpy="0 0 0"/>
+    <origin xyz="0 0 0" rpy="0 0 -1.5708"/>
     <geometry>
       <mesh filename="file://$(find medical_delivery_robot)/meshes/base_link.stl" scale="0.001 0.001 0.001"/>
@@ -18,9 +18,65 @@
   </visual>
   <collision>
-    <origin xyz="0 0 0" rpy="0 0 0"/>
+    <origin xyz="0 0 0" rpy="0 0 -1.5708"/>
     <geometry>
       <mesh filename="file://$(find medical_delivery_robot)/meshes/base_link.stl" scale="0.001 0.001 0.001"/>
     </geometry>
   </collision>
+</link>
+<link name="left_wheel_1">
+  <inertial>
+    <origin xyz="-0.03611520840332852 -7.184577711271973e-06 3.922141720499872e-07" rpy="0 0 0"/>
+    <mass value="7.769180436532471"/>
+    <inertia ixx="0.022657" iyy="0.013179" izz="0.013179" ixy="3e-06" iyz="0.0" ixz="-0.0"/>
+  </inertial>
+  <visual>
+    <origin xyz="0.17 0.003494 -0.059881" rpy="0 0 0"/>
+    <geometry>
+      <mesh filename="file://$(find medical_delivery_robot)/meshes/left_wheel_1.stl" scale="0.001 0.001 0.001"/>
+    </geometry>
+    <material name="silver"/>
+  </visual>
+  <collision>
+    <origin xyz="0.17 0.003494 -0.059881" rpy="0 0 0"/>
+    <geometry>
+      <mesh filename="file://$(find medical_delivery_robot)/meshes/left_wheel_1.stl" scale="0.001 0.001 0.001"/>
+    </geometry>
+  </collision>
+</link>
+<link name="right_wheel_1">
+  <inertial>
+    <origin xyz="0.03611520840332594 7.471004138964992e-06 3.9221417211243725e-07" rpy="0 0 0"/>
+    <mass value="7.769180436532471"/>
+    <inertia ixx="0.022657" iyy="0.013179" izz="0.013179" ixy="3e-06" iyz="-0.0" ixz="0.0"/>
+  </inertial>
+  <visual>
+    <origin xyz="-0.168 0.003494 -0.059881" rpy="0 0 0"/>
+    <geometry>
+      <mesh filename="file://$(find medical_delivery_robot)/meshes/right_wheel_1.stl" scale="0.001 0.001 0.001"/>
+    </geometry>
+    <material name="silver"/>
+  </visual>
+  <collision>
+    <origin xyz="-0.168 0.003494 -0.059881" rpy="0 0 0"/>
+    <geometry>
+      <mesh filename="file://$(find medical_delivery_robot)/meshes/right_wheel_1.stl" scale="0.001 0.001 0.001"/>
+    </geometry>
+  </collision>
+</link>
+<link name="imu_link">
+  <visual>
+    <geometry>
+      <box size="0.02 0.02 0.01"/>
+    </geometry>
+  </visual>
+  <collision>
+    <geometry>
+      <box size="0.02 0.02 0.01"/>
+    </geometry>
+  </collision>
+  <inertial>
+    <mass value="0.01"/>
+    <inertia ixx="1e-5" ixy="0" ixz="0" iyy="1e-5" iyz="0" izz="1e-5"/>
+  </inertial>
 </link>
 <link name="caster_wheel_1">
@@ -364,44 +420,4 @@
   </collision>
 </link>
-<link name="left_wheel_1">
-  <inertial>
-    <origin xyz="-0.03611520840332852 -7.184577711271973e-06 3.922141720499872e-07" rpy="0 0 0"/>
-    <mass value="7.769180436532471"/>
-    <inertia ixx="0.022657" iyy="0.013179" izz="0.013179" ixy="3e-06" iyz="0.0" ixz="-0.0"/>
-  </inertial>
-  <visual>
-    <origin xyz="0.17 0.003494 -0.059881" rpy="0 0 0"/>
-    <geometry>
-      <mesh filename="file://$(find medical_delivery_robot)/meshes/left_wheel_1.stl" scale="0.001 0.001 0.001"/>
-    </geometry>
-    <material name="silver"/>
-  </visual>
-  <collision>
-    <origin xyz="0.17 0.003494 -0.059881" rpy="0 0 0"/>
-    <geometry>
-      <mesh filename="file://$(find medical_delivery_robot)/meshes/left_wheel_1.stl" scale="0.001 0.001 0.001"/>
-    </geometry>
-  </collision>
-</link>
-<link name="right_wheel_1">
-  <inertial>
-    <origin xyz="0.03611520840332594 7.471004138964992e-06 3.9221417211243725e-07" rpy="0 0 0"/>
-    <mass value="7.769180436532471"/>
-    <inertia ixx="0.022657" iyy="0.013179" izz="0.013179" ixy="3e-06" iyz="-0.0" ixz="0.0"/>
-  </inertial>
-  <visual>
-    <origin xyz="-0.168 0.003494 -0.059881" rpy="0 0 0"/>
-    <geometry>
-      <mesh filename="file://$(find medical_delivery_robot)/meshes/right_wheel_1.stl" scale="0.001 0.001 0.001"/>
-    </geometry>
-    <material name="silver"/>
-  </visual>
-  <collision>
-    <origin xyz="-0.168 0.003494 -0.059881" rpy="0 0 0"/>
-    <geometry>
-      <mesh filename="file://$(find medical_delivery_robot)/meshes/right_wheel_1.stl" scale="0.001 0.001 0.001"/>
-    </geometry>
-  </collision>
-</link>
 <link name="front_cover_body_1">
   <inertial>
@@ -444,20 +460,4 @@
   </collision>
 </link>
-<link name="imu_link">
-  <visual>
-    <geometry>
-      <box size="0.02 0.02 0.01"/>
-    </geometry>
-  </visual>
-  <collision>
-    <geometry>
-      <box size="0.02 0.02 0.01"/>
-    </geometry>
-  </collision>
-  <inertial>
-    <mass value="0.01"/>
-    <inertia ixx="1e-5" ixy="0" ixz="0" iyy="1e-5" iyz="0" izz="1e-5"/>
-  </inertial>
-</link>
 <link name="lidar_camera_1">
   <inertial>
@@ -641,4 +641,21 @@
   </collision>
 </link>
+<joint name="left_wheel_joint" type="continuous">
+  <origin xyz="-0.003494 0.17 0.059881" rpy="0 0 -1.570796"/>
+  <parent link="base_link"/>
+  <child link="left_wheel_1"/>
+  <axis xyz="1.0 -0.0 0.0"/>
+</joint>
+<joint name="right_wheel_joint" type="continuous">
+  <origin xyz="-0.003494 -0.17 0.059881" rpy="0 0 -1.570796"/>
+  <parent link="base_link"/>
+  <child link="right_wheel_1"/>
+  <axis xyz="1.0 -0.0 0.0"/>
+</joint>
+<joint name="imu_joint" type="fixed">
+  <parent link="base_link"/>
+  <child link="imu_link"/>
+  <origin xyz="0 0 0.1" rpy="0 0 0"/>
+</joint>
 <joint name="Revolute 5" type="continuous">
   <origin xyz="0.0 0.0 0.0" rpy="0 0 0"/>
@@ -648,5 +665,5 @@
 </joint>
 <joint name="Revolute 7" type="continuous">
-  <origin xyz="0.179231 -0.20589 0.050881" rpy="0 0 0"/>
+  <origin xyz="0.2025 -0.17920 0.050881" rpy="0 0 0"/>
   <parent link="base_link"/>
   <child link="caster_wheel_plate_1"/>
@@ -680,5 +697,5 @@
 </joint>
 <joint name="Revolute 21" type="continuous">
-  <origin xyz="0.181711 0.199128 0.050881" rpy="0 0 0"/>
+  <origin xyz="0.2025 0.1770 0.050881" rpy="0 0 0"/>
   <parent link="base_link"/>
   <child link="caster_wheel_plate_2_1"/>
@@ -702,5 +719,5 @@
 </joint>
 <joint name="Revolute 25" type="continuous">
-  <origin xyz="-0.173289 0.199128 0.050881" rpy="0 0 0"/>
+  <origin xyz="-0.205 0.17750 0.050881" rpy="0 0 0"/>
   <parent link="base_link"/>
   <child link="caster_wheel_plate_3_1"/>
@@ -724,5 +741,5 @@
 </joint>
 <joint name="Revolute 29" type="continuous">
-  <origin xyz="-0.180769 -0.20589 0.050881" rpy="0 0 0"/>
+  <origin xyz="-0.205 -0.17750 0.050881" rpy="0 0 0"/>
   <parent link="base_link"/>
   <child link="caster_wheel_plate_4_1"/>
@@ -730,19 +747,7 @@
 </joint>
 <joint name="Rigid 30" type="fixed">
-  <origin xyz="0.239041 -0.18101 0.00666" rpy="0 0 0"/>
+  <origin xyz="-0.18101 -0.239041 0.00666" rpy="0 0 -1.570796"/>
   <parent link="base_link"/>
   <child link="middle_cover_body_1"/>
-</joint>
-<joint name="left_wheel_joint" type="continuous">
-  <origin xyz="-0.17 -0.003494 0.059881" rpy="0 0 0"/>
-  <parent link="base_link"/>
-  <child link="left_wheel_1"/>
-  <axis xyz="1.0 -0.0 0.0"/>
-</joint>
-<joint name="right_wheel_joint" type="continuous">
-  <origin xyz="0.168 -0.003494 0.059881" rpy="0 0 0"/>
-  <parent link="base_link"/>
-  <child link="right_wheel_1"/>
-  <axis xyz="1.0 -0.0 0.0"/>
 </joint>
 <joint name="Rigid 33" type="fixed">
@@ -771,9 +776,4 @@
   <origin xyz="0 0 0" rpy="-1.570796 0 -1.570796"/>
 </joint>
-<joint name="imu_joint" type="fixed">
-  <parent link="base_link"/>
-  <child link="imu_link"/>
-  <origin xyz="0 0 0.1" rpy="0 0 0"/>
-</joint>
 <joint name="Rigid 37" type="fixed">
   <origin xyz="-0.017313 0.264521 0.033" rpy="0 0 0"/>

Commit message: Add new world definition with random actor MaleVisitor1
- Created a new SDF world file 'random_actors.world'.
- Included sun and ground plane models.
- Defined an actor named 'MaleVisitor1' with a walking animation.
- Configured a trajectory for the actor with multiple waypoints.

File: urdf/medical_delivery.xacro (robot description, xacro)
@@ -4,4 +4,18 @@
 <xacro:include filename="$(find medical_delivery_robot)/urdf/medical_delivery.trans" />
 <xacro:include filename="$(find medical_delivery_robot)/urdf/medical_delivery.gazebo" />
+<!-- Base footprint for navigation and SLAM -->
+<link name="base_footprint">
+  <visual>
+    <origin xyz="0 0 0" rpy="0 0 0"/>
+    <geometry>
+      <box size="0.001 0.001 0.001"/>
+    </geometry>
+  </visual>
+</link>
+<joint name="base_footprint_joint" type="fixed">
+  <origin xyz="0 0 0.059881" rpy="0 0 0"/>
+  <parent link="base_footprint"/>
+  <child link="base_link"/>
+</joint>
 <link name="base_link">
   <inertial>
